Commit message: Deployed b3544352 to v6.4 with MkDocs 1.6.1 and mike 2.2.0

File: v6.4/assets/robots/piper/piper_v2.urdf (robot description, URDF)
Before this commit: robot piper_v2, 8 links, 7 joints
Links:
- removed link arm_base
- removed link gripper_center
- added link base_link, mass 1.02; collision mesh filename=package://piper_description/meshes/base_link.STL; visual mesh filename=package://piper_description/meshes/base_link.STL
- added link gripper_base, mass 0.45; collision mesh filename=package://piper_description/meshes/gripper_base.STL; visual mesh filename=package://piper_description/meshes/gripper_base.STL
- added link link7, mass 0.025; collision mesh filename=package://piper_description/meshes/link7.STL; visual mesh filename=package://piper_description/meshes/link7.STL
- added link link8, mass 0.025; collision mesh filename=package://piper_description/meshes/link8.STL; visual mesh filename=package://piper_description/meshes/link8.STL
- link link1: mass None -> 0.71; geometry collision mesh filename=package://piper_description/meshes/link1.STL; visual mesh filename=package://piper_description/meshes/link1.STL
- link link2: mass None -> 1.17; geometry collision mesh filename=package://piper_description/meshes/link2.STL; visual mesh filename=package://piper_description/meshes/link2.STL
- link link3: mass None -> 0.5; geometry collision mesh filename=package://piper_description/meshes/link3.STL; visual mesh filename=package://piper_description/meshes/link3.STL
- link link4: mass None -> 0.38; geometry collision mesh filename=package://piper_description/meshes/link4.STL; visual mesh filename=package://piper_description/meshes/link4.STL
- link link5: mass None -> 0.383; geometry collision mesh filename=package://piper_description/meshes/link5.STL; visual mesh filename=package://piper_description/meshes/link5.STL
- link link6: mass None -> 0.00699089613564366; geometry collision mesh filename=package://piper_description/meshes/link6.STL; visual mesh filename=package://piper_description/meshes/link6.STL
Joints:
- removed joint link6_to_gripper_center
- added joint joint6_to_gripper_base: type fixed, parent link6, child gripper_base, origin xyz=0 0 0 rpy=0 0 0
- added joint joint7: type prismatic, parent gripper_base, child link7, origin xyz=0 0 0.1358 rpy=1.5708 0 0, axis 0 0 1, limit lower=0 upper=0.035 effort=10 velocity=1
- added joint joint8: type prismatic, parent gripper_base, child link8, origin xyz=0 0 0.1358 rpy=1.5708 0 -3.1416, axis 0 0 -1, limit lower=-0.035 upper=0 effort=10 velocity=1
- joint joint1: limit lower=-2.6180 upper=2.6180 effort=100 velocity=5 -> lower=-2.618 upper=2.168 effort=100 velocity=5; origin xyz=0 0 0.123 rpy=0 0 -1.5708 -> xyz=0 0 0.123 rpy=0 0 0; parent arm_base -> base_link
- joint joint2: limit lower=0 upper=3.1416 effort=100 velocity=5 -> lower=0 upper=3.14 effort=100 velocity=5; origin xyz=0 0 0 rpy=1.5708 -0.034907 -1.5708 -> xyz=0 0 0 rpy=1.5708 -0.1359 -3.1416
- joint joint3: limit lower=-2.9671 upper=0 effort=100 velocity=5 -> lower=-2.967 upper=0 effort=100 velocity=5; origin xyz=0.28358 0.028726 0 rpy=0 0 0.06604341 -> xyz=0.28503 0 0 rpy=0 0 -1.7939
- joint joint4: limit lower=-1.6580 upper=1.6580 effort=100 velocity=5 -> lower=-1.745 upper=1.745 effort=100 velocity=5; origin xyz=-0.24221 0.068514 0 rpy=-1.5708 0 1.3826 -> xyz=-0.021984 -0.25075 0 rpy=1.5708 0 0
- joint joint5: limit lower=-1.8326 upper=1.8326 effort=100 velocity=5 -> lower=-1.22 upper=1.22 effort=100 velocity=5; origin xyz=0 0 0 rpy=1.5708 0 0 -> xyz=0 0 0 rpy=-1.5708 0 0
- joint joint6: limit lower=-2.7925 upper=2.7925 effort=100 velocity=5 -> lower=-2.0944 upper=2.0944 effort=100 velocity=3; origin xyz=0 0.091 0.0014165 rpy=-1.5708 -1.5708 0 -> xyz=8.8259E-05 -0.091 0 rpy=1.5708 0 0
