Commit message: Deployed b3544352 to v6.4 with MkDocs 1.6.1 and mike 2.2.0

File: v6.4/assets/robots/rizon4/flexiv_rizon4.urdf (robot description, URDF)
Before this commit: robot A02L-MP, 10 links, 9 joints
Links:
- link base_link: geometry collision mesh filename=meshes/collision/link0.stl; visual mesh filename=meshes/visual/link0.obj
- link link1: geometry collision mesh filename=meshes/collision/link1.stl; visual mesh filename=meshes/visual/link1.obj
- link link2: geometry collision mesh filename=meshes/collision/link2.stl; visual mesh filename=meshes/visual/link2.obj
- link link3: geometry collision mesh filename=meshes/collision/link3.stl; visual mesh filename=meshes/visual/link3.obj
- link link4: geometry collision mesh filename=meshes/collision/link4.stl; visual mesh filename=meshes/visual/link4.obj
- link link5: geometry collision mesh filename=meshes/collision/link5.stl; visual mesh filename=meshes/visual/link5.obj
- link link6: geometry collision mesh filename=meshes/collision/link6.stl; visual mesh filename=meshes/visual/link6.obj
- link link7: geometry collision mesh filename=meshes/collision/link7.stl; visual mesh filename=meshes/visual/link7.obj
