Commit message: Deployed b3544352 to v6.5 with MkDocs 1.6.1 and mike 2.2.0

File: v6.5/assets/robots/piper/piper_v2.urdf (robot description, URDF)
Before this commit: robot piper, 10 links, 9 joints
Links:
- link base_link: geometry collision mesh filename=./piper_description/meshes/base_link.STL; visual mesh filename=./piper_description/meshes/base_link.STL
- link gripper_base: geometry collision mesh filename=./piper_description/meshes/gripper_base.STL; visual mesh filename=./piper_description/meshes/gripper_base.STL
- link link1: geometry collision mesh filename=./piper_description/meshes/link1.STL; visual mesh filename=./piper_description/meshes/link1.STL
- link link2: geometry collision mesh filename=./piper_description/meshes/link2.STL; visual mesh filename=./piper_description/meshes/link2.STL
- link link3: geometry collision mesh filename=./piper_description/meshes/link3.STL; visual mesh filename=./piper_description/meshes/link3.STL
- link link4: geometry collision mesh filename=./piper_description/meshes/link4.STL; visual mesh filename=./piper_description/meshes/link4.STL
- link link5: geometry collision mesh filename=./piper_description/meshes/link5.STL; visual mesh filename=./piper_description/meshes/link5.STL
- link link6: geometry collision mesh filename=./piper_description/meshes/link6.STL; visual mesh filename=./piper_description/meshes/link6.STL
- link link7: geometry collision mesh filename=./piper_description/meshes/link7.STL; visual mesh filename=./piper_description/meshes/link7.STL
- link link8: geometry collision mesh filename=./piper_description/meshes/link8.STL; visual mesh filename=./piper_description/meshes/link8.STL

File: v6.5/assets/robots/ur16e/ur16e.urdf (robot description, URDF)
Before this commit: robot ur16e, 12 links, 11 joints
Links:
- link base_link_inertia: geometry collision mesh filename=./ur_description/meshes/ur10e/collision/base.stl; visual mesh filename=./ur_description/meshes/ur10e/visual/base.dae
- link forearm_link: geometry collision mesh filename=./ur_description/meshes/ur16e/collision/forearm.stl; visual mesh filename=./ur_description/meshes/ur16e/visual/forearm.dae
- link shoulder_link: geometry collision mesh filename=./ur_description/meshes/ur10e/collision/shoulder.stl; visual mesh filename=./ur_description/meshes/ur10e/visual/shoulder.dae
- link upper_arm_link: geometry collision mesh filename=./ur_description/meshes/ur16e/collision/upperarm.stl; visual mesh filename=./ur_description/meshes/ur16e/visual/upperarm.dae
- link wrist_1_link: geometry collision mesh filename=./ur_description/meshes/ur10e/collision/wrist1.stl; visual mesh filename=./ur_description/meshes/ur10e/visual/wrist1.dae
- link wrist_2_link: geometry collision mesh filename=./ur_description/meshes/ur10e/collision/wrist2.stl; visual mesh filename=./ur_description/meshes/ur10e/visual/wrist2.dae
- link wrist_3_link: geometry collision mesh filename=./ur_description/meshes/ur10e/collision/wrist3.stl; visual mesh filename=./ur_description/meshes/ur10e/visual/wrist3.dae

File: v6.5/assets/robots/ur5e/ur5e.urdf (robot description, URDF)
Before this commit: robot ur5e, 12 links, 11 joints
Links:
- link base_link_inertia: geometry collision mesh filename=./ur_description/meshes/ur5e/collision/base.stl; visual mesh filename=./ur_description/meshes/ur5e/visual/base.dae
- link forearm_link: geometry collision mesh filename=./ur_description/meshes/ur5e/collision/forearm.stl; visual mesh filename=./ur_description/meshes/ur5e/visual/forearm.dae
- link shoulder_link: geometry collision mesh filename=./ur_description/meshes/ur5e/collision/shoulder.stl; visual mesh filename=./ur_description/meshes/ur5e/visual/shoulder.dae
- link upper_arm_link: geometry collision mesh filename=./ur_description/meshes/ur5e/collision/upperarm.stl; visual mesh filename=./ur_description/meshes/ur5e/visual/upperarm.dae
- link wrist_1_link: geometry collision mesh filename=./ur_description/meshes/ur5e/collision/wrist1.stl; visual mesh filename=./ur_description/meshes/ur5e/visual/wrist1.dae
- link wrist_2_link: geometry collision mesh filename=./ur_description/meshes/ur5e/collision/wrist2.stl; visual mesh filename=./ur_description/meshes/ur5e/visual/wrist2.dae
- link wrist_3_link: geometry collision mesh filename=./ur_description/meshes/ur5e/collision/wrist3.stl; visual mesh filename=./ur_description/meshes/ur5e/visual/wrist3.dae
